File: zavrsni/zavrsni.kicad_pcb (KiCad board)
At the start: 2 copper layers, 149.4 x 96.2 mm, 60 parts, among them Q1 BC337, Q2 BC327, U1 CS4335, U2 WeAct STM32F411CEU6 v3.0, U3 NE5532, U4 TL074, U5 LM358, U6 LM317_TO-220, U7 UC1609C LCD Board

Commit message: ST7920, CS4271, new project direction
Parts:
- removed Jin1, Jout1, Jvcc1, Jvss1: Conn_01x01_Pin, Connector_Wire:SolderWirePad_1x01_SMD_4x8mm
- removed Q1: BC337, Package_TO_SOT_THT:TO-92_Inline
- removed Q2: BC327, Package_TO_SOT_THT:TO-92_Inline
- removed RV1: R_Potentiometer_MountingPin, ljepi:pot vertikalni 5 pin
- removed SW_DOWN1, SW_OK1, SW_PRESET_0, SW_PRESET_1, SW_PRESET_2, SW_PRESET_3, SW_TUNER1, SW_UP1: SW_Push, Button_Switch_THT:SW_PUSH_6mm_H13mm
- added C10: 10u, Capacitor_THT:CP_Radial_D5.0mm_P2.50mm, F.Cu at (109.7, 114.5)
- added C16: 100n, Capacitor_THT:C_Disc_D5.0mm_W2.5mm_P5.00mm, F.Cu at (102.5, 143.5)
- added C17: 100n, Capacitor_THT:C_Disc_D5.0mm_W2.5mm_P5.00mm, F.Cu at (102.5, 147.5)
- added C23: 100n, Capacitor_THT:C_Disc_D5.0mm_W2.5mm_P5.00mm, F.Cu at (102.5, 151.6)
- added C25: 100n, Capacitor_THT:C_Disc_D5.0mm_W2.5mm_P5.00mm, F.Cu at (102.5, 155.6)
- added DS1: AG12864E, ljepi:LCD_12864-21M_V1.5, F.Cu at (17.0, 90.0)
- added JIN1: Conn_01x01_Pin, Connector_Wire:SolderWirePad_1x01_SMD_4x8mm, F.Cu at (271.8, 21.4)
- added R14: 22k, Resistor_THT:R_Axial_DIN0207_L6.3mm_D2.5mm_P2.54mm_Vertical, F.Cu at (116.2, 137.1)
- added R15: 10k, Resistor_THT:R_Axial_DIN0207_L6.3mm_D2.5mm_P2.54mm_Vertical, F.Cu at (116.2, 141.2)
- added R16: 15k, Resistor_THT:R_Axial_DIN0207_L6.3mm_D2.5mm_P5.08mm_Vertical, F.Cu at (128.5, 144.3)
- added R17: 22k, Resistor_THT:R_Axial_DIN0207_L6.3mm_D2.5mm_P2.54mm_Vertical, F.Cu at (122.4, 125.0)
- added R18: 22k, Resistor_THT:R_Axial_DIN0207_L6.3mm_D2.5mm_P2.54mm_Vertical, F.Cu at (122.4, 129.0)
- added R19: 22k, Resistor_THT:R_Axial_DIN0207_L6.3mm_D2.5mm_P2.54mm_Vertical, F.Cu at (122.4, 133.1)
- added R20: 22k, Resistor_THT:R_Axial_DIN0207_L6.3mm_D2.5mm_P2.54mm_Vertical, F.Cu at (122.4, 137.1)
- added R21: 680, Resistor_THT:R_Axial_DIN0207_L6.3mm_D2.5mm_P5.08mm_Vertical, F.Cu at (128.5, 148.3)
- added R22: 470k, Resistor_THT:R_Axial_DIN0207_L6.3mm_D2.5mm_P2.54mm_Vertical, F.Cu at (122.4, 141.2)
- added R23: 33, Resistor_THT:R_Axial_DIN0207_L6.3mm_D2.5mm_P5.08mm_Vertical, F.Cu at (128.5, 152.4)
- added R5: 470k, Resistor_THT:R_Axial_DIN0207_L6.3mm_D2.5mm_P2.54mm_Vertical, F.Cu at (285.8, 80.8)
- added SW1: EC11, ljepi:ec11, F.Cu at (244.5, 68.1)
- added U8: TL072, Package_DIP:DIP-8_W7.62mm, F.Cu at (126.6, 113.3)
- C1: value 15n -> 10n
- C11, C12: value 100n -> 220p; footprint Capacitor_THT:C_Disc_D5.0mm_W2.5mm_P5.00mm -> Capacitor_THT:C_Disc_D5.0mm_W2.5mm_P2.50mm
- C13: value 10u -> 10n; footprint Capacitor_THT:CP_Radial_D5.0mm_P2.50mm -> Capacitor_THT:C_Disc_D5.0mm_W2.5mm_P2.50mm
- C2, C22, C24: value 10u -> 1u
- C4: value 10u -> 100n; footprint Capacitor_THT:CP_Radial_D5.0mm_P2.50mm -> Capacitor_THT:C_Disc_D5.0mm_W2.5mm_P5.00mm
- C5: value 680u -> 100n; footprint Capacitor_THT:CP_Radial_D8.0mm_P2.50mm -> Capacitor_THT:C_Disc_D5.0mm_W2.5mm_P5.00mm
- C8: value 100n -> 10u; footprint Capacitor_THT:C_Disc_D5.0mm_W2.5mm_P5.00mm -> Capacitor_THT:CP_Radial_D5.0mm_P2.50mm
- C9: value 680u -> 47u; footprint Capacitor_THT:CP_Radial_D8.0mm_P2.50mm -> Capacitor_THT:CP_Radial_D5.0mm_P2.50mm
- R1: value 300 -> 680
- R10, R11, R3, R4: value 10k -> 51k
- R12: value 1k -> 33k; footprint Resistor_THT:R_Axial_DIN0207_L6.3mm_D2.5mm_P5.08mm_Vertical -> Resistor_THT:R_Axial_DIN0207_L6.3mm_D2.5mm_P2.54mm_Vertical
- R13: value 1k -> 33k
- R2, R6: value 300 -> 22k
- U1: value CS4335 -> TL072; footprint Package_SO:SOIC-8_3.9x4.9mm_P1.27mm -> Package_DIP:DIP-8_W7.62mm
- U3: value NE5532 -> TL072; footprint Package_DIP:DIP-8_W7.62mm_Socket -> Package_DIP:DIP-8_W7.62mm
- U4: footprint Package_DIP:DIP-14_W7.62mm_Socket -> Package_DIP:DIP-14_W7.62mm
- U5: value LM358 -> TL074; footprint Package_DIP:DIP-8_W7.62mm_Socket -> Package_DIP:DIP-14_W7.62mm
- U7: value UC1609C LCD Board -> CS4271; footprint ljepi:PinSocket1x9_66mm_x_26mm -> Package_SO:TSSOP-28_4.4x9.7mm_P0.65mm
- moved R8 233.0 mm to (285.8, 93.0), turned to 0 degrees
- moved R7 230.0 mm to (285.8, 88.9), turned to 0 degrees
- moved R1 229.4 mm to (281.5, 45.7)
- moved C6 227.5 mm to (273.4, 48.4), turned to 0 degrees
- moved C1 222.6 mm to (271.0, 28.2), turned to 0 degrees
- moved C21 219.8 mm to (270.6, 101.0), turned to 0 degrees
- moved C19 219.3 mm to (279.3, 97.7), turned to 0 degrees
- moved C20 217.6 mm to (279.3, 104.2), turned to 0 degrees
- moved R10 217.4 mm to (281.5, 53.8), turned to 0 degrees
- moved R11 217.3 mm to (285.8, 97.0), turned to 0 degrees
- moved D1 214.4 mm to (282.0, 18.5), turned to 0 degrees
- moved R6 213.8 mm to (285.8, 84.8)
- moved D2 212.8 mm to (282.0, 22.3), turned to 0 degrees
- moved C14 211.8 mm to (270.6, 88.9), turned to 0 degrees
- moved R9 209.6 mm to (281.5, 49.7), turned to 0 degrees
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Connections:
- C1 pad 1: Net-(C1-Pad1) -> Net-(U4A-+)
- C11 pad 1: +12V -> Net-(U4A--)
- C11 pad 2: +0V -> Net-(C11-Pad2)
- C12 pad 1: /LCD_VCC -> Net-(U8B-+)
- C12 pad 2: GNDREF -> Net-(C12-Pad2)
- C13 pad 1: /LCD_VCC -> Net-(U3A-+)
- C14 pad 1: +12V -> VCC
- C15 pad 1: Net-(U4B-+) -> /VADC_BIAS
- C15 pad 2: GNDREF -> GNDPWR
- C18 pad 2: GNDREF -> GNDPWR
- C19 pad 2: GNDREF -> GNDPWR
- C2 pad 1: Net-(C1-Pad1) -> Net-(U7-VQ1)
- C2 pad 2: Net-(U3B-+) -> GNDPWR
- C20 pad 2: GNDREF -> GNDPWR
- C21 pad 1: Net-(U5A-+) -> Net-(U1A-+)
- C21 pad 2: +0V -> GNDPWR
- C22 pad 1: +12V -> +3V3
- C22 pad 2: +0V -> GNDPWR
- C24 pad 1: +12V -> +5V
- C24 pad 2: +0V -> GNDPWR
- C3 pad 1: +5V -> Net-(JIN1-Pin_1)
- C3 pad 2: GNDREF -> /IN
- C4 pad 1: +5V -> GNDREF
- C4 pad 2: GNDREF -> GNDPWR
- C5 pad 1: +12V -> Net-(U7-VQ1)
- C5 pad 2: GNDREF -> GNDPWR
- C6 pad 2: +0V -> GNDPWR
- C7 pad 1: Net-(C7-Pad1) -> Net-(U5A--)
- C7 pad 2: Net-(C7-Pad2) -> Net-(U7-AINA)
- C8 pad 1: +12V -> Net-(U7-AOUTA-)
- C8 pad 2: +0V -> Net-(C8-Pad2)
- C9 pad 1: +12V -> Net-(U7-FILT+)
- C9 pad 2: +0V -> GNDPWR
- R1 pad 1: Net-(U3A--) -> Net-(U1B--)
- R1 pad 2: Net-(C1-Pad1) -> Net-(U4A-+)
- R10 pad 1: Net-(U4B-+) -> /VADC_BIAS
- R10 pad 2: +5V -> +3V3
- R11 pad 1: GNDREF -> GNDPWR
- R11 pad 2: Net-(U4B-+) -> /VADC_BIAS
- R12 pad 1: Net-(U4B--) -> Net-(U4C-+)
- R12 pad 2: Net-(C7-Pad2) -> GNDPWR
- R13 pad 1: Net-(R13-Pad1) -> VCC
- R13 pad 2: Net-(U4B--) -> Net-(U4D-+)
- R2 pad 1: GNDREF -> VCC
- R2 pad 2: Net-(U3B-+) -> Net-(U4C-+)
- R3 pad 1: Net-(U5A-+) -> Net-(U1A-+)
- R3 pad 2: +12V -> VCC
- R4 pad 1: +0V -> GNDPWR
- R4 pad 2: Net-(U5A-+) -> Net-(U1A-+)
- R6 pad 1: Net-(U3B--) -> Net-(U4A--)
- R9 pad 2: Net-(R13-Pad1) -> Net-(C11-Pad2)
- U1 pad 1: /DAC_DAT -> GNDREF
- U1 pad 2: /DAC_BCLK -> GNDREF
- U1 pad 3: /DAC_LRCLK -> Net-(U1A-+)
- U1 pad 4: /DAC_MCLK -> (no net)
- U1 pad 5: /OUT -> /IN
- U1 pad 6: GNDREF -> Net-(U1B--)
- U1 pad 7: +5V -> Net-(U1B--)
- U1 pad 8: unconnected-(U1-AOUTL-Pad8) -> (no net)
- U2 pad 1: /DAC_LRCLK -> unconnected-(U2-B12-Pad1)
- U2 pad 10: /BTN_OK -> unconnected-(U2-A15-Pad10)
- U2 pad 11: /BTN_DOWN -> unconnected-(U2-B3-Pad11)
- U2 pad 12: /BTN_PRESET3 -> unconnected-(U2-B4-Pad12)
- U2 pad 13: /BTN_PRESET2 -> unconnected-(U2-B5-Pad13)
- U2 pad 14: /BTN_PRESET1 -> unconnected-(U2-B6-Pad14)
- U2 pad 15: /BTN_PRESET0 -> unconnected-(U2-B7-Pad15)
- U2 pad 16: /BTN_UP -> unconnected-(U2-B8-Pad16)
- U2 pad 17: /BTN_TUNER -> unconnected-(U2-B9-Pad17)
- U2 pad 19: GNDREF -> GNDPWR
- U2 pad 2: /DAC_BCLK -> unconnected-(U2-B13-Pad2)
- U2 pad 26: /ADC_IN -> unconnected-(U2-A0-Pad26)
- U2 pad 29: /DAC_MCLK -> unconnected-(U2-A3-Pad29)
- U2 pad 31: /LCD_SCK -> unconnected-(U2-A5-Pad31)
- U2 pad 32: /LCD_RST -> unconnected-(U2-A6-Pad32)
- U2 pad 33: /LCD_SDA -> unconnected-(U2-A7-Pad33)
- U2 pad 34: /LCD_CS -> unconnected-(U2-B0-Pad34)
- U2 pad 35: /LCD_CD -> unconnected-(U2-B1-Pad35)
- U2 pad 36: /LCD_VCC -> unconnected-(U2-B2-Pad36)
- U2 pad 39: GNDREF -> GNDPWR
- U2 pad 4: /DAC_DAT -> unconnected-(U2-B15-Pad4)
- U3 pad 3: /IN -> Net-(U3A-+)
- U3 pad 4: +0V -> (no net)
- U3 pad 5: Net-(U3B-+) -> (no net)
- U3 pad 6: Net-(U3B--) -> (no net)
- U3 pad 7: Net-(C7-Pad1) -> (no net)
- U3 pad 8: +12V -> (no net)
- U4 pad 1: Net-(D2-A) -> Net-(C11-Pad2)
- U4 pad 10: GNDREF -> Net-(U4C-+)
- U4 pad 11: +0V -> (no net)
- U4 pad 12: Net-(D1-A) -> Net-(U4D-+)
- U4 pad 13: /ADC_IN -> Net-(D1-A)
- U4 pad 14: /ADC_IN -> Net-(D2-A)
- U4 pad 2: Net-(D1-A) -> Net-(U4A--)
- U4 pad 3: +5V -> Net-(U4A-+)
- U4 pad 4: +12V -> (no net)
- U4 pad 5: Net-(U4B-+) -> (no net)
- U4 pad 6: Net-(U4B--) -> (no net)
- U4 pad 7: Net-(R13-Pad1) -> (no net)
- U5 pad 1: Net-(Q1-B) -> Net-(U5A--)
- U5 pad 2: Net-(Q1-B) -> Net-(U5A--)
- U5 pad 3: Net-(U5A-+) -> Net-(D1-A)
- U5 pad 4: +0V -> (no net)
- U5 pad 8: +12V -> (no net)
- U6 pad 3: +12V -> VCC
- U7 pad 1: GNDREF -> unconnected-(U7-XTO-Pad1)
- U7 pad 2: +3V3 -> GNDPWR
- U7 pad 3: GNDREF -> /MCU.MCLK
- U7 pad 4: /LCD_VCC -> /MCU.LRCK
- U7 pad 5: /LCD_SCK -> /MCU.SCLK
- U7 pad 6: /LCD_SDA -> /MCU.ADC_OUT
- U7 pad 7: /LCD_RST -> /MCU.DAC_IN
- U7 pad 8: /LCD_CD -> GNDPWR
- U7 pad 9: /LCD_CS -> +3V3
Routing:
- net /BTN_PRESET0: track 137.2 -> 0.00 mm, vias 2 -> 0
- net /BTN_PRESET3: track 135.3 -> 0.00 mm, vias 2 -> 0
- net /BTN_TUNER: track 121.6 -> 0.00 mm, vias 2 -> 0
- net /BTN_OK: track 114.5 -> 0.00 mm, vias 2 -> 0
- net /BTN_PRESET2: track 111.8 -> 0.00 mm, vias 2 -> 0
- net /BTN_PRESET1: track 111.1 -> 0.00 mm, vias 2 -> 0
- net +5V: track 97.6 -> 0.00 mm
- net /BTN_UP: track 95.6 -> 0.00 mm, vias 2 -> 0
- net +0V: track 93.1 -> 0.00 mm, vias 2 -> 0
- net /BTN_DOWN: track 91.1 -> 0.00 mm, vias 2 -> 0
- net +12V: track 79.6 -> 0.00 mm
- net /LCD_SCK: track 67.0 -> 0.00 mm
- net /LCD_SDA: track 55.3 -> 0.00 mm
- net /DAC_MCLK: track 46.1 -> 0.00 mm, vias 1 -> 0
- net Net-(D1-A): track 38.9 -> 0.00 mm
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- removed copper zone on F.Cu, net +0V
- removed copper zone on F.Cu, net +12V
- removed copper zone on F.Cu, net GNDREF
Other:
- board size 149.4 x 96.2 mm -> 175 x 85 mm
- board text removed: "${CRTAO} Mutliefekt pedala za električnu gitaru ${DATUM} v${VERZIJA}"

Commit message: Updated buttons and switched to I2S for the codec.
Parts:
- removed DS1: AG12864E, ljepi:LCD_12864-21M_V1.5
- removed JIN1: Conn_01x01_Pin, Connector_Wire:SolderWirePad_1x01_SMD_4x8mm
- added J1: Barrel_Jack_MountingPin, Connector_BarrelJack:BarrelJack_Horizontal, F.Cu at (163.8, 103.4)
- added J2: SameSky 6.35 horizontal jack, ljepi:6.35 horizontalni 4pin samesky, F.Cu at (62.1, 106.2)
- added J3: USB_B, Connector_USB:USB_B_Lumberg_2411_02_Horizontal, F.Cu at (141.7, 87.0)
- added J4: SameSky 6.35 horizontal jack, ljepi:6.35 horizontalni 4pin samesky, F.Cu at (62.1, 122.2)
- added R24: 22k, Resistor_THT:R_Axial_DIN0207_L6.3mm_D2.5mm_P2.54mm_Vertical, F.Cu at (107.2, 124.4)
- added R25: 22k, Resistor_THT:R_Axial_DIN0207_L6.3mm_D2.5mm_P2.54mm_Vertical, F.Cu at (113.4, 100.1)
- added R26: 22k, Resistor_THT:R_Axial_DIN0207_L6.3mm_D2.5mm_P2.54mm_Vertical, F.Cu at (113.4, 104.1)
- added R27: 22k, Resistor_THT:R_Axial_DIN0207_L6.3mm_D2.5mm_P2.54mm_Vertical, F.Cu at (113.4, 108.2)
- added R28: 680, Resistor_THT:R_Axial_DIN0207_L6.3mm_D2.5mm_P5.08mm_Vertical, F.Cu at (119.5, 132.5)
- added R29: 470k, Resistor_THT:R_Axial_DIN0207_L6.3mm_D2.5mm_P2.54mm_Vertical, F.Cu at (113.4, 112.2)
- added SW_BNK+1: SW_Push, Button_Switch_THT:SW_PUSH_6mm_H7.3mm, F.Cu at (82.4, 100.1)
- added SW_BNK-1: SW_Push, Button_Switch_THT:SW_PUSH_6mm_H7.3mm, F.Cu at (82.4, 108.6)
- added SW_PRE+1: SW_Push, Button_Switch_THT:SW_PUSH_6mm_H7.3mm, F.Cu at (82.4, 117.2)
- added SW_PRE-1: SW_Push, Button_Switch_THT:SW_PUSH_6mm_H7.3mm, F.Cu at (82.4, 125.7)
- added SW_VOL+1: SW_Push, Button_Switch_THT:SW_PUSH_6mm_H7.3mm, F.Cu at (82.4, 134.3)
- added SW_VOL-1: SW_Push, Button_Switch_THT:SW_PUSH_6mm_H7.3mm, F.Cu at (82.4, 142.8)
- added U10: TL072, Package_DIP:DIP-8_W7.62mm, F.Cu at (149.3, 122.1)
- added U9: TL072, Package_DIP:DIP-8_W7.62mm, F.Cu at (138.5, 122.1)
- C1: value 10n -> 100n; footprint Capacitor_THT:C_Disc_D5.0mm_W2.5mm_P2.50mm -> Capacitor_THT:C_Disc_D5.0mm_W2.5mm_P5.00mm
- C11: value 220p -> 100n; footprint Capacitor_THT:C_Disc_D5.0mm_W2.5mm_P2.50mm -> Capacitor_THT:C_Disc_D5.0mm_W2.5mm_P5.00mm
- C12: value 220p -> 10u; footprint Capacitor_THT:C_Disc_D5.0mm_W2.5mm_P2.50mm -> Capacitor_THT:CP_Radial_D5.0mm_P2.50mm
- C13: value 10n -> 1u; footprint Capacitor_THT:C_Disc_D5.0mm_W2.5mm_P2.50mm -> Capacitor_THT:CP_Radial_D5.0mm_P2.50mm
- C14: value 100n -> 47u; footprint Capacitor_THT:C_Disc_D5.0mm_W2.5mm_P5.00mm -> Capacitor_THT:CP_Radial_D5.0mm_P2.50mm
- C17, C18: value 100n -> 1u; footprint Capacitor_THT:C_Disc_D5.0mm_W2.5mm_P5.00mm -> Capacitor_THT:CP_Radial_D5.0mm_P2.50mm
- C19, C7: value 10u -> 100n; footprint Capacitor_THT:CP_Radial_D5.0mm_P2.50mm -> Capacitor_THT:C_Disc_D5.0mm_W2.5mm_P5.00mm
- C2: value 1u -> 100n; footprint Capacitor_THT:CP_Radial_D5.0mm_P2.50mm -> Capacitor_THT:C_Disc_D5.0mm_W2.5mm_P5.00mm
- C20: value 100u -> 100n; footprint Capacitor_THT:CP_Radial_D5.0mm_P2.50mm -> Capacitor_THT:C_Disc_D5.0mm_W2.5mm_P5.00mm
- C21: value 100n -> 10u; footprint Capacitor_THT:C_Disc_D5.0mm_W2.5mm_P5.00mm -> Capacitor_THT:CP_Radial_D5.0mm_P2.50mm
- C22: value 1u -> 10u
- C23: value 100n -> 220p; footprint Capacitor_THT:C_Disc_D5.0mm_W2.5mm_P5.00mm -> Capacitor_THT:C_Disc_D5.0mm_W2.5mm_P2.50mm
- C24: value 1u -> 10n; footprint Capacitor_THT:CP_Radial_D5.0mm_P2.50mm -> Capacitor_THT:C_Disc_D5.0mm_W2.5mm_P2.50mm
- C3: value 100n -> 680u; footprint Capacitor_THT:C_Disc_D5.0mm_W2.5mm_P5.00mm -> Capacitor_THT:CP_Radial_D8.0mm_P2.50mm
- C6: value 680u -> 10n; footprint Capacitor_THT:CP_Radial_D8.0mm_P2.50mm -> Capacitor_THT:C_Disc_D5.0mm_W2.5mm_P2.50mm
- C8: value 10u -> 220p; footprint Capacitor_THT:CP_Radial_D5.0mm_P2.50mm -> Capacitor_THT:C_Disc_D5.0mm_W2.5mm_P2.50mm
- C9: value 47u -> 100u
- H1, H2, H3, H4: footprint MountingHole:MountingHole_4.3mm_M4_ISO7380_Pad -> MountingHole:MountingHole_3.2mm_M3_Pad
- R1: value 680 -> 51k; footprint Resistor_THT:R_Axial_DIN0207_L6.3mm_D2.5mm_P5.08mm_Vertical -> Resistor_THT:R_Axial_DIN0207_L6.3mm_D2.5mm_P10.16mm_Horizontal
- R10: value 51k -> 33k; footprint Resistor_THT:R_Axial_DIN0207_L6.3mm_D2.5mm_P5.08mm_Vertical -> Resistor_THT:R_Axial_DIN0207_L6.3mm_D2.5mm_P2.54mm_Vertical
- R11: value 51k -> 1k; footprint Resistor_THT:R_Axial_DIN0207_L6.3mm_D2.5mm_P2.54mm_Vertical -> Resistor_THT:R_Axial_DIN0207_L6.3mm_D2.5mm_P5.08mm_Vertical
- R12: value 33k -> 22k
- R14: value 22k -> 33k
- R15: value 10k -> 22k
- R16: value 15k -> 33
- R17, R19, R20: value 22k -> 33; footprint Resistor_THT:R_Axial_DIN0207_L6.3mm_D2.5mm_P2.54mm_Vertical -> Resistor_THT:R_Axial_DIN0207_L6.3mm_D2.5mm_P5.08mm_Vertical
- R18: value 22k -> 10k
- R2: value 22k -> 51k; footprint Resistor_THT:R_Axial_DIN0207_L6.3mm_D2.5mm_P2.54mm_Vertical -> Resistor_THT:R_Axial_DIN0207_L6.3mm_D2.5mm_P10.16mm_Horizontal
- R21: value 680 -> 10k; footprint Resistor_THT:R_Axial_DIN0207_L6.3mm_D2.5mm_P5.08mm_Vertical -> Resistor_THT:R_Axial_DIN0207_L6.3mm_D2.5mm_P2.54mm_Vertical
- R22: value 470k -> 33; footprint Resistor_THT:R_Axial_DIN0207_L6.3mm_D2.5mm_P2.54mm_Vertical -> Resistor_THT:R_Axial_DIN0207_L6.3mm_D2.5mm_P5.08mm_Vertical
- R23: value 33 -> 10k; footprint Resistor_THT:R_Axial_DIN0207_L6.3mm_D2.5mm_P5.08mm_Vertical -> Resistor_THT:R_Axial_DIN0207_L6.3mm_D2.5mm_P2.54mm_Vertical
- R3: value 51k -> 470k; footprint Resistor_THT:R_Axial_DIN0207_L6.3mm_D2.5mm_P10.16mm_Horizontal -> Resistor_THT:R_Axial_DIN0207_L6.3mm_D2.5mm_P2.54mm_Vertical
- R4: value 51k -> 3k3; footprint Resistor_THT:R_Axial_DIN0207_L6.3mm_D2.5mm_P10.16mm_Horizontal -> Resistor_THT:R_Axial_DIN0207_L6.3mm_D2.5mm_P2.54mm_Vertical
- R5: value 470k -> 10k
- R6: value 22k -> 680; footprint Resistor_THT:R_Axial_DIN0207_L6.3mm_D2.5mm_P2.54mm_Vertical -> Resistor_THT:R_Axial_DIN0207_L6.3mm_D2.5mm_P5.08mm_Vertical
- R7: value 3k3 -> 22k
- R8: value 10k -> 15k; footprint Resistor_THT:R_Axial_DIN0207_L6.3mm_D2.5mm_P2.54mm_Vertical -> Resistor_THT:R_Axial_DIN0207_L6.3mm_D2.5mm_P5.08mm_Vertical
- R9: value 1k -> 20k; footprint Resistor_THT:R_Axial_DIN0207_L6.3mm_D2.5mm_P5.08mm_Vertical -> Resistor_THT:R_Axial_DIN0207_L6.3mm_D2.5mm_P2.54mm_Vertical
- U2: value WeAct STM32F411CEU6 v3.0 -> LM317_TO-220; footprint Package_DIP:DIP-40_W15.24mm_Socket -> Package_TO_SOT_THT:TO-220-3_Horizontal_TabDown
- U3: value TL072 -> LM317_TO-220; footprint Package_DIP:DIP-8_W7.62mm -> Package_TO_SOT_THT:TO-220-3_Horizontal_TabDown
- U5: value TL074 -> ~; footprint Package_DIP:DIP-14_W7.62mm -> ljepi:LCD_12864-21M_V1.5
- U6: value LM317_TO-220 -> WeAct STM32F411CEU6 v3.0; footprint Package_TO_SOT_THT:TO-220-3_Horizontal_TabDown -> Package_DIP:DIP-40_W15.24mm_Socket
- U7: value CS4271 -> TL074; footprint Package_SO:TSSOP-28_4.4x9.7mm_P0.65mm -> Package_DIP:DIP-14_W7.62mm
- U8: value TL072 -> CS4271; footprint Package_DIP:DIP-8_W7.62mm -> Package_SO:TSSOP-28_4.4x9.7mm_P0.65mm
- moved D1 235.7 mm to (75.4, 131.9)
- moved D2 235.7 mm to (75.4, 135.7)
- moved C14 222.9 mm to (53.6, 139.8)
- moved C21 213.9 mm to (60.2, 139.8)
- moved C3 213.7 mm to (68.5, 146.1)
- moved C18 213.5 mm to (60.2, 133.3)
- moved U5 206.7 mm to (45.6, 97.3)
- moved C1 192.5 mm to (92.5, 100.1)
- moved R10 192.3 mm to (101.1, 120.3)
- moved R9 192.3 mm to (101.1, 116.3)
- moved C19 190.0 mm to (92.5, 132.5)
- moved C20 189.6 mm to (92.5, 136.5)
- moved R5 186.7 mm to (101.1, 108.2)
- moved R7 186.2 mm to (101.1, 112.2)
- moved C15 180.8 mm to (92.5, 124.4)
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Connections:
- C1 pad 1: Net-(U4A-+) -> Net-(U1A-+)
- C1 pad 2: GNDREF -> GNDPWR
- C10 pad 1: Net-(U7-AOUTA+) -> +3V3
- C10 pad 2: Net-(C10-Pad2) -> GNDPWR
- C11 pad 1: Net-(U4A--) -> +3V3
- C11 pad 2: Net-(C11-Pad2) -> GNDPWR
- C12 pad 1: Net-(U8B-+) -> Net-(U7A--)
- C12 pad 2: Net-(C12-Pad2) -> Net-(U8-AINA)
- C13 pad 1: Net-(U3A-+) -> +3V3
- C13 pad 2: GNDREF -> GNDPWR
- C14 pad 1: VCC -> Net-(U8-FILT+)
- C14 pad 2: GNDREF -> GNDPWR
- C15 pad 1: /VADC_BIAS -> Net-(U8-FILT+)
- C16 pad 1: Net-(U3A--) -> +3V3
- C16 pad 2: /OUT -> GNDPWR
- C17 pad 1: Net-(U7-FILT+) -> +5V
- C18 pad 1: +3V3 -> Net-(U8-VQ1)
- C19 pad 1: +3V3 -> +5V
- C2 pad 1: Net-(U7-VQ1) -> GNDREF
- C20 pad 1: +3V3 -> Net-(U8-VQ1)
- C21 pad 1: Net-(U1A-+) -> Net-(U8-AOUTA-)
- C21 pad 2: GNDPWR -> Net-(C21-Pad2)
- C22 pad 1: +3V3 -> Net-(U8-AOUTA+)
- C22 pad 2: GNDPWR -> Net-(C22-Pad2)
- C23 pad 1: +3V3 -> Net-(U9B-+)
- C23 pad 2: GNDPWR -> Net-(C23-Pad2)
- C24 pad 1: +5V -> Net-(U10A-+)
- C24 pad 2: GNDPWR -> GNDREF
- C25 pad 1: +5V -> Net-(U10A--)
- C25 pad 2: GNDPWR -> Net-(C25-Pad2)
- C3 pad 1: Net-(JIN1-Pin_1) -> GNDREF
- C3 pad 2: /IN -> GNDPWR
- C4 pad 1: GNDREF -> Net-(C4-Pad1)
- C4 pad 2: GNDPWR -> /IN
- C5 pad 1: Net-(U7-VQ1) -> VCC
- C6 pad 1: GNDREF -> Net-(U4A-+)
- C6 pad 2: GNDPWR -> GNDREF
- C7 pad 1: Net-(U5A--) -> +5V
- C7 pad 2: Net-(U7-AINA) -> GNDPWR
- C8 pad 1: Net-(U7-AOUTA-) -> Net-(U4A--)
- C9 pad 1: Net-(U7-FILT+) -> +3V3
- H1 pad 1: GNDREF -> GNDPWR
- H2 pad 1: GNDREF -> GNDPWR
- H3 pad 1: GNDREF -> GNDPWR
- H4 pad 1: GNDREF -> GNDPWR
- R1 pad 1: Net-(U1B--) -> Net-(U1A-+)
- R1 pad 2: Net-(U4A-+) -> VCC
- R10 pad 1: /VADC_BIAS -> Net-(U3-ADJ)
- R10 pad 2: +3V3 -> GNDPWR
- R11 pad 1: GNDPWR -> Net-(D1-A)
- R11 pad 2: /VADC_BIAS -> Net-(C8-Pad2)
- R12 pad 1: Net-(U4C-+) -> VCC
- R12 pad 2: GNDPWR -> Net-(U4C-+)
- R13 pad 1: VCC -> Net-(U4C-+)
- R13 pad 2: Net-(U4D-+) -> GNDPWR
- R14 pad 1: Net-(U4D-+) -> VCC
- R14 pad 2: GNDPWR -> Net-(U4D-+)
- R15 pad 1: Net-(U7-AINA) -> Net-(U4D-+)
- R15 pad 2: /VREF_ADC -> GNDPWR
- R16 pad 1: Net-(U4A--) -> /MCU.SCLK
- R16 pad 2: Net-(C11-Pad2) -> Net-(U6-B13)
- R17 pad 1: Net-(C10-Pad2) -> /MCU.LRCK
- R17 pad 2: Net-(U8B--) -> Net-(U6-B12)
- R18 pad 1: GNDREF -> Net-(U8-AINA)
- R18 pad 2: Net-(U8B--) -> /VREF_ADC
- R19 pad 1: Net-(U8B-+) -> /MCU.MCLK
- R19 pad 2: Net-(C8-Pad2) -> /MCU.MCLK0
- R2 pad 1: VCC -> GNDPWR
- R2 pad 2: Net-(U4C-+) -> Net-(U1A-+)
- R20 pad 1: Net-(C12-Pad2) -> Net-(U8-SDOUT)
- R20 pad 2: Net-(U8B-+) -> /MCU.ADC_OUT
- R21 pad 1: Net-(C12-Pad2) -> GNDPWR
- R21 pad 2: Net-(U3A-+) -> /MCU.RST
- R22 pad 1: GNDPWR -> Net-(U8-SDIN)
- R22 pad 2: /OUT -> /MCU.DAC_IN
- R23 pad 1: unconnected-(R23-Pad1) -> +3V3
- R23 pad 2: /MCU.MCLK -> Net-(U8-I2S/L~{J})
- R3 pad 1: Net-(U1A-+) -> GNDREF
- R3 pad 2: VCC -> /IN
- R4 pad 1: GNDPWR -> +5V
- R4 pad 2: Net-(U1A-+) -> Net-(U2-ADJ)
- R5 pad 1: GNDREF -> Net-(U2-ADJ)
- R5 pad 2: /IN -> GNDPWR
- R6 pad 1: Net-(U4A--) -> Net-(U1B--)
- R6 pad 2: GNDREF -> Net-(U4A-+)
- R7 pad 1: +5V -> Net-(U4A--)
- R7 pad 2: Net-(U6-ADJ) -> GNDREF
- R8 pad 1: Net-(U6-ADJ) -> Net-(U4A--)
- R8 pad 2: GNDREF -> Net-(C8-Pad2)
- R9 pad 1: Net-(D1-A) -> +3V3
- R9 pad 2: Net-(C11-Pad2) -> Net-(U3-ADJ)
- SW1 pad A: unconnected-(SW1-PadA) -> Net-(U6-C14)
- SW1 pad B: unconnected-(SW1-PadB) -> Net-(U6-C13)
- SW1 pad C: unconnected-(SW1-PadC) -> GNDPWR
- SW1 pad MP: unconnected-(SW1-PadMP) -> GNDPWR
- SW1 pad S1: unconnected-(SW1-PadS1) -> Net-(U6-C15)
- SW1 pad S2: unconnected-(SW1-PadS2) -> GNDPWR
- U2 pad 1: unconnected-(U2-B12-Pad1) -> Net-(U2-ADJ)
- U2 pad 2: unconnected-(U2-B13-Pad2) -> +5V
- U2 pad 3: unconnected-(U2-B14-Pad3) -> VCC
- U3 pad 1: Net-(U3A--) -> Net-(U3-ADJ)
- U3 pad 2: Net-(U3A--) -> +3V3
- U3 pad 3: Net-(U3A-+) -> +5V
- U4 pad 1: Net-(C11-Pad2) -> Net-(C8-Pad2)
- U5 pad 1: Net-(U5A--) -> GNDPWR
- U5 pad 10: (no net) -> unconnected-(U5-DB3-Pad10)
- U5 pad 11: (no net) -> unconnected-(U5-DB4-Pad11)
- U5 pad 12: (no net) -> unconnected-(U5-DB5-Pad12)
- U5 pad 13: (no net) -> unconnected-(U5-DB6-Pad13)
- U5 pad 14: (no net) -> unconnected-(U5-DB7-Pad14)
- U5 pad 2: Net-(U5A--) -> +3V3
- U5 pad 3: Net-(D1-A) -> unconnected-(U5-VO-Pad3)
- U5 pad 4: (no net) -> /LCD.CS
- U5 pad 5: (no net) -> /LCD.DAT
- U5 pad 6: (no net) -> /LCD.CLK
- U5 pad 7: (no net) -> unconnected-(U5-DB0-Pad7)
- U5 pad 8: (no net) -> unconnected-(U5-DB1-Pad8)
- U5 pad 9: (no net) -> unconnected-(U5-DB2-Pad9)
- U6 pad 1: Net-(U6-ADJ) -> Net-(U6-B12)
- U6 pad 2: +5V -> Net-(U6-B13)
- U6 pad 3: VCC -> /MCU.ADC_OUT
- U7 pad 1: unconnected-(U7-XTO-Pad1) -> Net-(U7A--)
- U7 pad 10: +3V3 -> (no net)
- U7 pad 11: GNDPWR -> (no net)
- U7 pad 12: GNDPWR -> (no net)
- U7 pad 13: unconnected-(U7-I2S/L~{J}-Pad13) -> (no net)
- U7 pad 14: /MCU.RST -> (no net)
- U7 pad 2: GNDPWR -> Net-(U7A--)
- U7 pad 3: /MCU.MCLK -> Net-(D1-A)
- U7 pad 4: /MCU.LRCK -> (no net)
- U7 pad 5: /MCU.SCLK -> (no net)
- U7 pad 6: /MCU.ADC_OUT -> (no net)
- U7 pad 7: /MCU.DAC_IN -> (no net)
- U7 pad 8: GNDPWR -> (no net)
- U7 pad 9: +3V3 -> (no net)
- U8 pad 1: /VREF_ADC -> unconnected-(U8-XTO-Pad1)
- U8 pad 2: /VREF_ADC -> GNDPWR
- U8 pad 3: Net-(U7-VQ1) -> /MCU.MCLK
- U8 pad 4: (no net) -> /MCU.LRCK
- U8 pad 5: Net-(U8B-+) -> /MCU.SCLK
- U8 pad 6: Net-(U8B--) -> Net-(U8-SDOUT)
- U8 pad 7: Net-(C12-Pad2) -> Net-(U8-SDIN)
- U8 pad 8: (no net) -> GNDPWR
Other:
- board outline removed

Commit message: KiCad 10
Parts:
- removed R21: 10k, Resistor_THT:R_Axial_DIN0207_L6.3mm_D2.5mm_P2.54mm_Vertical
- removed U10: TL072, Package_DIP:DIP-8_W7.62mm
- added C26: 10u, Capacitor_THT:CP_Radial_D5.0mm_P2.50mm, F.Cu at (-101.3, 121.7)
- added C27: 10u, Capacitor_THT:CP_Radial_D5.0mm_P2.50mm, F.Cu at (-101.3, 128.2)
- C1: value 100n -> 47u; footprint Capacitor_THT:C_Disc_D5.0mm_W2.5mm_P5.00mm -> Capacitor_THT:CP_Radial_D5.0mm_P2.50mm
- C3: value 680u -> 10u; footprint Capacitor_THT:CP_Radial_D8.0mm_P2.50mm -> Capacitor_THT:CP_Radial_D5.0mm_P2.50mm
- R1, R2: value 51k -> 10k
- SW_BNK+1, SW_BNK-1, SW_PRE+1, SW_PRE-1, SW_VOL+1, SW_VOL-1: footprint Button_Switch_THT:SW_PUSH_6mm_H7.3mm -> Button_Switch_THT:SW_PUSH_6mm_H13mm
- U1: value TL072 -> TL074; footprint Package_DIP:DIP-8_W7.62mm -> Package_DIP:DIP-14_W7.62mm
- U9: value TL072 -> LM358
- moved J1 305.0 mm to (-137.7, 149.2)
- moved C23 300.1 mm to (-133.2, 153.9)
- moved C24 300.1 mm to (-133.2, 158.0)
- moved C6 300.1 mm to (-133.2, 145.8)
- moved C8 300.1 mm to (-133.2, 149.9)
- moved R11 278.8 mm to (-158.9, 122.0)
- moved R16 278.8 mm to (-158.9, 126.0)
- moved R17 278.8 mm to (-158.9, 130.1)
- moved R19 278.8 mm to (-158.9, 134.1)
- moved R20 278.8 mm to (-158.9, 138.2)
- moved R22 278.8 mm to (-158.9, 142.2)
- moved R28 278.8 mm to (-158.9, 146.3)
- moved R6 278.8 mm to (-158.9, 113.9)
- moved R8 278.8 mm to (-158.9, 117.9)
- moved H1 275.8 mm to (-92.8, 135.2)
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Connections:
- C1 pad 1: Net-(U1A-+) -> GNDREF
- C12 pad 1: Net-(U7A--) -> Net-(U4B--)
- C18 pad 1: Net-(U8-VQ1) -> Net-(U4C-+)
- C20 pad 1: Net-(U8-VQ1) -> Net-(U4C-+)
- C23 pad 1: Net-(U9B-+) -> Net-(U4D--)
- C24 pad 1: Net-(U10A-+) -> Net-(U7A-+)
- C25 pad 1: Net-(U10A--) -> Net-(U7A--)
- C3 pad 1: GNDREF -> Net-(U9A-+)
- C6 pad 1: Net-(U4A-+) -> Net-(U1C-+)
- C8 pad 1: Net-(U4A--) -> Net-(U1C--)
- J1 pad 3: (no net) -> GNDPWR
- R1 pad 1: Net-(U1A-+) -> Net-(U9A-+)
- R12 pad 2: Net-(U4C-+) -> Net-(U1D-+)
- R13 pad 1: Net-(U4C-+) -> Net-(U1D-+)
- R14 pad 2: Net-(U4D-+) -> Net-(U4A-+)
- R15 pad 1: Net-(U4D-+) -> Net-(U4A-+)
- R2 pad 2: Net-(U1A-+) -> Net-(U9A-+)
- R24 pad 2: Net-(U9B--) -> Net-(U4D-+)
- R25 pad 1: Net-(U9B-+) -> Net-(U4D--)
- R26 pad 2: Net-(U9B--) -> Net-(U4D-+)
- R27 pad 2: Net-(U9B-+) -> Net-(U4D--)
- R28 pad 2: Net-(U10A-+) -> Net-(U7A-+)
- R6 pad 2: Net-(U4A-+) -> Net-(U1C-+)
- R7 pad 1: Net-(U4A--) -> Net-(U1C--)
- R8 pad 1: Net-(U4A--) -> Net-(U1C--)
- U1 pad 1: GNDREF -> (no net)
- U1 pad 2: GNDREF -> (no net)
- U1 pad 3: Net-(U1A-+) -> (no net)
- U1 pad 4: (no net) -> unconnected-(U1E-V+-Pad4)
- U1 pad 8: (no net) -> Net-(C8-Pad2)
- U4 pad 1: Net-(C8-Pad2) -> Net-(D2-A)
- U4 pad 11: (no net) -> unconnected-(U4E-V--Pad11)
- U4 pad 13: Net-(D1-A) -> Net-(U4D--)
- U4 pad 14: Net-(D2-A) -> Net-(C23-Pad2)
- U4 pad 2: Net-(U4A--) -> Net-(D1-A)
- U4 pad 4: (no net) -> unconnected-(U4E-V+-Pad4)
- U4 pad 5: (no net) -> Net-(D1-A)
- U4 pad 6: (no net) -> Net-(U4B--)
- U4 pad 7: (no net) -> Net-(U4B--)
- U4 pad 8: Net-(D1-K) -> /VREF_ADC
- U4 pad 9: Net-(D1-A) -> /VREF_ADC
- U7 pad 3: Net-(D1-A) -> Net-(U7A-+)
- U8 pad 15: Net-(U8-VQ1) -> Net-(U4C-+)
- U9 pad 1: /VREF_ADC -> GNDREF
- U9 pad 2: /VREF_ADC -> GNDREF
- U9 pad 3: Net-(U8-VQ1) -> Net-(U9A-+)
- U9 pad 4: (no net) -> unconnected-(U9C-V--Pad4)
- U9 pad 5: Net-(U9B-+) -> Net-(U9A-+)
- U9 pad 7: Net-(C23-Pad2) -> Net-(U9B--)
- U9 pad 8: (no net) -> unconnected-(U9C-V+-Pad8)
Routing:
- added copper zone on B.Cu, net GNDPWR
Other:
- board outline added: 183 x 130 mm
