File: zavrsni/zavrsni.kicad_pcb (KiCad board)
At the start: 2 copper layers, 183 x 130 mm, 81 parts, among them J1 Barrel_Jack_MountingPin, J2 SameSky 6.35 horizontal jack, J3 USB_B, J4 SameSky 6.35 horizontal jack, SW1 EC11, U1 TL074, U2 LM317_TO-220, U3 LM317_TO-220, U4 TL074, U6 WeAct STM32F411CEU6 v3.0, U7 TL074, U8 CS4271, U9 LM358

Commit message: Started work on the PCB. Started drawing the codec/STM32 part of the layout.
Parts:
- removed J2, J4: SameSky 6.35 horizontal jack, ljepi:6.35 horizontalni 4pin samesky
- removed U4: TL074, Package_DIP:DIP-14_W7.62mm
- added C28: 10u, Capacitor_THT:CP_Radial_D5.0mm_P2.50mm, F.Cu at (30.9, 104.0)
- added C29: 100n, Capacitor_THT:C_Disc_D5.0mm_W2.5mm_P5.00mm, F.Cu at (30.9, 76.4)
- added C30: 100n, Capacitor_THT:C_Disc_D5.0mm_W2.5mm_P5.00mm, F.Cu at (30.9, 80.4)
- added C31: 100n, Capacitor_THT:C_Disc_D5.0mm_W2.5mm_P5.00mm, F.Cu at (30.9, 84.5)
- added C32: 100u, Capacitor_THT:CP_Radial_D5.0mm_P2.50mm, F.Cu at (30.9, 110.5)
- added C33: 100n, Capacitor_THT:C_Disc_D5.0mm_W2.5mm_P5.00mm, F.Cu at (84.9, 183.6)
- added D3: LED, LED_THT:LED_D3.0mm, F.Cu at (-29.4, 105.4)
- added D4: LED, LED_THT:LED_D3.0mm, F.Cu at (-29.4, 110.9)
- added D5: LED, LED_THT:LED_D3.0mm, F.Cu at (-29.4, 116.4)
- added D6: LED, LED_THT:LED_D3.0mm, F.Cu at (-29.4, 121.8)
- added D7: LED, LED_THT:LED_D3.0mm, F.Cu at (-29.4, 127.3)
- added D8: LED, LED_THT:LED_D3.0mm, F.Cu at (-29.4, 132.8)
- added JIN1: SameSky 6.35 horizontal jack, ljepi:6.35 horizontalni 4pin samesky, F.Cu at (94.0, 147.3)
- added JOUT1: SameSky 6.35 horizontal jack, ljepi:6.35 horizontalni 4pin samesky, F.Cu at (132.0, 189.4)
- added JP_LIM1: SolderJumper_2_Open, Jumper:SolderJumper-2_P1.3mm_Open_RoundedPad1.0x1.5mm, F.Cu at (133.6, 144.2)
- added R21: 100, Resistor_THT:R_Axial_DIN0207_L6.3mm_D2.5mm_P5.08mm_Vertical, F.Cu at (-29.0, 92.6)
- added R30: 1k, Resistor_THT:R_Axial_DIN0207_L6.3mm_D2.5mm_P2.54mm_Vertical, F.Cu at (-8.05, 116.4)
- added R31: 1k, Resistor_THT:R_Axial_DIN0207_L6.3mm_D2.5mm_P2.54mm_Vertical, F.Cu at (-1.91, 96.2)
- added R32: 1k, Resistor_THT:R_Axial_DIN0207_L6.3mm_D2.5mm_P2.54mm_Vertical, F.Cu at (-1.91, 100.2)
- added R33: 1k, Resistor_THT:R_Axial_DIN0207_L6.3mm_D2.5mm_P2.54mm_Vertical, F.Cu at (-1.91, 104.3)
- added R34: 1k, Resistor_THT:R_Axial_DIN0207_L6.3mm_D2.5mm_P2.54mm_Vertical, F.Cu at (-1.91, 108.3)
- added R35: 1k, Resistor_THT:R_Axial_DIN0207_L6.3mm_D2.5mm_P2.54mm_Vertical, F.Cu at (-1.91, 112.4)
- added TP_3V3: Conn_01x01, Connector_PinHeader_2.54mm:PinHeader_1x01_P2.54mm_Vertical, F.Cu at (26.1, 116.1)
- added TP_5V1: Conn_01x01, Connector_PinHeader_2.54mm:PinHeader_1x01_P2.54mm_Vertical, F.Cu at (26.1, 120.7)
- added TP_CODEC1: Conn_01x05, Connector_PinHeader_2.54mm:PinHeader_1x05_P2.54mm_Vertical, F.Cu at (210.6, 151.9)
- added TP_FILT1: Conn_01x01, Connector_PinHeader_2.54mm:PinHeader_1x01_P2.54mm_Vertical, F.Cu at (150.2, 136.0)
- added TP_LIM1: Conn_01x01, Connector_PinHeader_2.54mm:PinHeader_1x01_P2.54mm_Vertical, F.Cu at (26.1, 129.8)
- added TP_OUT1: Conn_01x02, Connector_PinHeader_2.54mm:PinHeader_1x02_P2.54mm_Vertical, F.Cu at (150.9, 121.5)
- added U10: TL072, Package_DIP:DIP-8_W7.62mm, F.Cu at (95.7, 171.9)
- R16, R19: footprint Resistor_THT:R_Axial_DIN0207_L6.3mm_D2.5mm_P5.08mm_Vertical -> Resistor_THT:R_Axial_DIN0207_L6.3mm_D2.5mm_P10.16mm_Horizontal
- R17: footprint Resistor_THT:R_Axial_DIN0207_L6.3mm_D2.5mm_P5.08mm_Vertical -> Resistor_THT:R_Axial_DIN0207_L6.3mm_D2.5mm_P15.24mm_Horizontal
- R22: footprint Resistor_THT:R_Axial_DIN0207_L6.3mm_D2.5mm_P5.08mm_Vertical -> Resistor_THT:R_Axial_DIN0207_L6.3mm_D2.5mm_P2.54mm_Vertical
- R23: footprint Resistor_THT:R_Axial_DIN0207_L6.3mm_D2.5mm_P2.54mm_Vertical -> Resistor_THT:R_Axial_DIN0207_L6.3mm_D2.5mm_P5.08mm_Vertical
- U6: footprint Package_DIP:DIP-40_W15.24mm_Socket -> ljepi:STM32F411CEU6 WeAct V3.0
- U7: value TL074 -> TL072; footprint Package_DIP:DIP-14_W7.62mm -> Package_DIP:DIP-8_W7.62mm
- moved R19 322.7 mm to (160.7, 89.5)
- moved R17 318.0 mm to (158.2, 107.1), turned to 180 degrees
- moved C15 317.6 mm to (150.1, 132.7)
- moved R16 315.2 mm to (155.5, 104.1), turned to 180 degrees
- moved R20 310.4 mm to (150.6, 114.7), turned to 90 degrees
- moved C19 310.2 mm to (142.4, 129.4)
- moved C16 308.3 mm to (139.8, 113.4)
- moved R22 307.6 mm to (147.4, 113.6), turned to 90 degrees
- moved C20 305.2 mm to (137.3, 130.5), turned to 180 degrees
- moved C14 258.1 mm to (150.1, 128.8)
- moved C12 256.2 mm to (141.6, 138.8), turned to 90 degrees
- moved C17 252.3 mm to (144.3, 133.7)
- moved C18 245.3 mm to (137.3, 126.2), turned to 180 degrees
- moved U6 245.1 mm to (167.0, 93.6), turned to 90 degrees
- moved C13 241.6 mm to (129.2, 161.5)
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Connections:
- C12 pad 1: Net-(U4B--) -> Net-(U7A--)
- C18 pad 1: Net-(U4C-+) -> Net-(U7B-+)
- C20 pad 1: Net-(U4C-+) -> Net-(U7B-+)
- C24 pad 1: Net-(U7A-+) -> Net-(U10B-+)
- C25 pad 1: Net-(U7A--) -> Net-(U10B--)
- C6 pad 1: Net-(U1C-+) -> Net-(U1B-+)
- C8 pad 1: Net-(U1C--) -> Net-(U1B--)
- R1 pad 2: VCC -> VCCA
- R12 pad 1: VCC -> VCCA
- R12 pad 2: Net-(U1D-+) -> Net-(U1C-+)
- R13 pad 1: Net-(U1D-+) -> Net-(U1C-+)
- R14 pad 1: VCC -> VCCA
- R14 pad 2: Net-(U4A-+) -> Net-(U1D-+)
- R15 pad 1: Net-(U4A-+) -> Net-(U1D-+)
- R28 pad 2: Net-(U7A-+) -> Net-(U10B-+)
- R6 pad 1: Net-(U1B--) -> Net-(U1A--)
- R6 pad 2: Net-(U1C-+) -> Net-(U1B-+)
- R7 pad 1: Net-(U1C--) -> Net-(U1B--)
- R8 pad 1: Net-(U1C--) -> Net-(U1B--)
- U1 pad 1: (no net) -> Net-(U1A--)
- U1 pad 11: unconnected-(U1E-V--Pad11) -> GNDPWR
- U1 pad 14: Net-(D1-K) -> Net-(D2-A)
- U1 pad 2: (no net) -> Net-(U1A--)
- U1 pad 3: (no net) -> /IN
- U1 pad 4: unconnected-(U1E-V+-Pad4) -> VCC
- U1 pad 5: /IN -> Net-(U1B-+)
- U1 pad 7: Net-(U1B--) -> Net-(C8-Pad2)
- U1 pad 8: Net-(C8-Pad2) -> Net-(D1-K)
- U1 pad 9: Net-(U1C--) -> Net-(D1-A)
- U7 pad 3: Net-(U7A-+) -> Net-(JP_LIM1-B)
- U7 pad 4: (no net) -> GNDPWR
- U7 pad 5: (no net) -> Net-(U7B-+)
- U7 pad 6: (no net) -> /VREF_ADC
- U7 pad 7: (no net) -> /VREF_ADC
- U7 pad 8: (no net) -> VCC
- U8 pad 15: Net-(U4C-+) -> Net-(U7B-+)
- U9 pad 4: unconnected-(U9C-V--Pad4) -> GNDPWR
- U9 pad 8: unconnected-(U9C-V+-Pad8) -> VCC
Routing:
- net /MCU.MCLK: track 0.00 -> 71.4 mm
- net /MCU.RST: track 0.00 -> 40.7 mm
- net /MCU.SCLK: track 0.00 -> 23.9 mm
- net /MCU.LRCK: track 0.00 -> 22.8 mm
- net /VREF_ADC: track 0.00 -> 22.0 mm
- net GNDPWR: track 0.00 -> 21.7 mm
- net /MCU.DAC_IN: track 0.00 -> 18.4 mm
- net Net-(TP_FILT1-Pin_1): track 0.00 -> 15.2 mm
- net Net-(U7A--): track 0.00 -> 15.2 mm
- net Net-(U8-AINA): track 0.00 -> 11.9 mm
- net /MCU.ADC_OUT: track 0.00 -> 10.5 mm
- net +3V3: track 0.00 -> 10.5 mm
- net Net-(TP_CODEC1-Pin_4): track 0.00 -> 9.69 mm
- net Net-(U7B-+): track 0.00 -> 9.22 mm
- net +5V: track 0.00 -> 9.16 mm
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- added copper zone on F.Cu, net +3V3
- added copper zone on F.Cu, net GNDPWR
- added copper zone on F.Cu, net Net-(U8-AINA)

Commit message: PCB almost done.
Parts:
- removed D3, D4, D5, D6, D7, D8: LED, LED_THT:LED_D3.0mm
- removed R30, R31, R32, R33, R34, R35: 1k, Resistor_THT:R_Axial_DIN0207_L6.3mm_D2.5mm_P2.54mm_Vertical
- removed TP_3V3, TP_5V1: Conn_01x01, Connector_PinHeader_2.54mm:PinHeader_1x01_P2.54mm_Vertical
- removed TP_CODEC1: Conn_01x05, Connector_PinHeader_2.54mm:PinHeader_1x05_P2.54mm_Vertical
- added J2: Conn_01x05, Connector_PinHeader_2.54mm:PinHeader_1x05_P2.54mm_Vertical, F.Cu at (153.1, 105.1)
- added JP_3V3: SolderJumper_2_Open, Jumper:SolderJumper-2_P1.3mm_Open_RoundedPad1.0x1.5mm, F.Cu at (128.5, 98.2)
- added JP_5V1: SolderJumper_2_Open, Jumper:SolderJumper-2_P1.3mm_Open_RoundedPad1.0x1.5mm, F.Cu at (110.2, 99.9)
- R25: footprint Resistor_THT:R_Axial_DIN0207_L6.3mm_D2.5mm_P2.54mm_Vertical -> Resistor_THT:R_Axial_DIN0207_L6.3mm_D2.5mm_P10.16mm_Horizontal
- R26: footprint Resistor_THT:R_Axial_DIN0207_L6.3mm_D2.5mm_P2.54mm_Vertical -> Resistor_THT:R_Axial_DIN0207_L6.3mm_D2.5mm_P7.62mm_Horizontal
- R3: footprint Resistor_THT:R_Axial_DIN0207_L6.3mm_D2.5mm_P2.54mm_Vertical -> Resistor_THT:R_Axial_DIN0207_L6.3mm_D2.5mm_P5.08mm_Vertical
- R6: footprint Resistor_THT:R_Axial_DIN0207_L6.3mm_D2.5mm_P5.08mm_Vertical -> Resistor_THT:R_Axial_DIN0207_L6.3mm_D2.5mm_P7.62mm_Horizontal
- R8: footprint Resistor_THT:R_Axial_DIN0207_L6.3mm_D2.5mm_P5.08mm_Vertical -> Resistor_THT:R_Axial_DIN0207_L6.3mm_D2.5mm_P2.54mm_Vertical
- U2, U3: footprint Package_TO_SOT_THT:TO-220-3_Horizontal_TabDown -> Package_TO_SOT_THT:TO-220-3_Vertical
- moved R28 194.1 mm to (161.0, 140.2), turned to -90 degrees
- moved R29 190.7 mm to (179.8, 145.1), turned to -90 degrees
- moved R27 181.4 mm to (171.7, 132.9), turned to 180 degrees
- moved R25 180.4 mm to (170.1, 128.6), turned to 180 degrees
- moved R24 173.3 mm to (161.5, 132.3)
- moved R26 170.8 mm to (157.8, 145.1), turned to 90 degrees
- moved R11 160.6 mm to (120.1, 132.0), turned to -90 degrees
- moved R8 160.3 mm to (114.4, 139.8)
- moved C25 159.9 mm to (172.0, 147.5)
- moved R18 157.4 mm to (141.2, 137.6), turned to 180 degrees
- moved R6 156.6 mm to (103.9, 147.0)
- moved R9 142.6 mm to (121.5, 98.0), turned to -90 degrees
- moved R10 142.6 mm to (121.7, 103.8), turned to -90 degrees
- moved C23 142.5 mm to (172.8, 127.3), turned to -90 degrees
- moved J3 140.6 mm to (23.1, 185.5)
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Connections:
- net Net-(TP_CODEC1-Pin_4) renamed /MCU.ADC_OUT0
- net Net-(TP_CODEC1-Pin_5) renamed /MCU.DAC_IN0
- net Net-(U6-B12) renamed /MCU.LRCK0
- net Net-(U6-B13) renamed /MCU.SCLK0
- R4 pad 1: +5V -> Net-(JP_5V1-A)
- R9 pad 1: +3V3 -> Net-(JP_3V3-A)
- SW1 pad S1: Net-(U6-C15) -> GNDPWR
- SW1 pad S2: GNDPWR -> Net-(U6-C15)
- U2 pad 2: +5V -> Net-(JP_5V1-A)
- U3 pad 2: +3V3 -> +5V
- U3 pad 3: +5V -> Net-(JP_3V3-A)
- U6 pad 12: /BTN.BNK- -> /BTN.PRE-
- U6 pad 13: /BTN.BNK+ -> /BTN.PRE+
- U6 pad 16: /BTN.PRE- -> /BTN.BNK-
- U6 pad 17: /BTN.PRE+ -> /BTN.BNK+
- U6 pad 20: +3V3 -> unconnected-(U6-3V3-Pad20)
Routing:
- net VCC: track 0.00 -> 217.2 mm, vias 0 -> 6
- net /BTN.BNK-: track 0.00 -> 67.7 mm, vias 0 -> 2
- net +5V: track 9.16 -> 75.9 mm, vias 0 -> 2
- net Net-(D1-A): track 0.00 -> 57.2 mm, vias 0 -> 2
- net Net-(U6-C15): track 0.00 -> 53.4 mm
- net +3V3: track 10.5 -> 53.6 mm, vias 0 -> 2
- net /BTN.VOL+: track 0.00 -> 40.3 mm
- net /BTN.BNK+: track 0.00 -> 38.3 mm
- net Net-(U6-C14): track 0.00 -> 37.1 mm
- net Net-(U6-C13): track 0.00 -> 36.1 mm
- net /BTN.VOL-: track 0.00 -> 24.7 mm
- net Net-(C23-Pad2): track 0.00 -> 19.9 mm
- net Net-(U10A-+): track 0.00 -> 15.4 mm
- net Net-(U1B-+): track 0.00 -> 14.2 mm
- net Net-(C4-Pad1): track 0.00 -> 13.9 mm
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- added copper zone on F.Cu, net GNDREF
Other:
- copper layers 2 -> 4

Commit message: PCB done. Code, PCB screw holes and 3D design left
Parts:
- removed C18: 1u, Capacitor_THT:CP_Radial_D5.0mm_P2.50mm
- removed U9: LM358, Package_DIP:DIP-8_W7.62mm
- added R30: 22?, Resistor_THT:R_Axial_DIN0207_L6.3mm_D2.5mm_P15.24mm_Horizontal, F.Cu at (135.3, 102.5)
- added R31: 22?, Resistor_THT:R_Axial_DIN0207_L6.3mm_D2.5mm_P7.62mm_Horizontal, F.Cu at (141.3, 105.6)
- added R32: 150, Resistor_THT:R_Axial_DIN0411_L9.9mm_D3.6mm_P12.70mm_Horizontal, F.Cu at (105.0, 68.5)
- added U4: TL072, Package_DIP:DIP-8_W7.62mm, F.Cu at (171.0, 67.6)
- J3: footprint Connector_USB:USB_B_Lumberg_2411_02_Horizontal -> ljepi:USB B Female
- R1, R19: footprint Resistor_THT:R_Axial_DIN0207_L6.3mm_D2.5mm_P10.16mm_Horizontal -> Resistor_THT:R_Axial_DIN0207_L6.3mm_D2.5mm_P15.24mm_Horizontal
- R10: footprint Resistor_THT:R_Axial_DIN0207_L6.3mm_D2.5mm_P2.54mm_Vertical -> Resistor_THT:R_Axial_DIN0207_L6.3mm_D2.5mm_P5.08mm_Vertical
- R16, R2, R25: footprint Resistor_THT:R_Axial_DIN0207_L6.3mm_D2.5mm_P10.16mm_Horizontal -> Resistor_THT:R_Axial_DIN0207_L6.3mm_D2.5mm_P2.54mm_Vertical
- R17: footprint Resistor_THT:R_Axial_DIN0207_L6.3mm_D2.5mm_P15.24mm_Horizontal -> Resistor_THT:R_Axial_DIN0207_L6.3mm_D2.5mm_P2.54mm_Vertical
- R18: footprint Resistor_THT:R_Axial_DIN0207_L6.3mm_D2.5mm_P2.54mm_Vertical -> Resistor_THT:R_Axial_DIN0207_L6.3mm_D2.5mm_P10.16mm_Horizontal
- R20, R23, R28, R3: footprint Resistor_THT:R_Axial_DIN0207_L6.3mm_D2.5mm_P5.08mm_Vertical -> Resistor_THT:R_Axial_DIN0207_L6.3mm_D2.5mm_P2.54mm_Vertical
- R21: footprint Resistor_THT:R_Axial_DIN0207_L6.3mm_D2.5mm_P5.08mm_Vertical -> Resistor_THT:R_Axial_DIN0207_L6.3mm_D2.5mm_P7.62mm_Horizontal
- R26: footprint Resistor_THT:R_Axial_DIN0207_L6.3mm_D2.5mm_P7.62mm_Horizontal -> Resistor_THT:R_Axial_DIN0207_L6.3mm_D2.5mm_P5.08mm_Vertical
- moved R1 214.4 mm to (181.3, 70.8), turned to 180 degrees
- moved R2 212.3 mm to (178.7, 73.9)
- moved R21 198.4 mm to (167.8, 67.6), turned to 90 degrees
- moved C3 178.8 mm to (181.3, 78.2), turned to 180 degrees
- moved C1 174.2 mm to (172.3, 51.3)
- moved C7 172.2 mm to (186.4, 129.8), turned to -90 degrees
- moved C28 166.6 mm to (149.2, 76.4), turned to 180 degrees
- moved J1 164.8 mm to (202.5, 31.7), turned to -90 degrees
- moved C10 158.0 mm to (108.3, 98.0), turned to -90 degrees
- moved C32 149.4 mm to (200.4, 49.3), turned to 180 degrees
- moved H3 149.2 mm to (24.8, 147.8)
- moved H4 149.2 mm to (24.8, 155.7)
- moved C11 146.6 mm to (164.8, 116.4), turned to 180 degrees
- moved JIN1 138.6 mm to (168.9, 30.6), turned to -90 degrees
- moved C29 136.3 mm to (165.6, 55.8), turned to 90 degrees
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Connections:
- C12 pad 1: Net-(U7A--) -> Net-(TP_LIM1-Pin_1)
- C12 pad 2: Net-(U8-AINA) -> Net-(JP_LIM1-A)
- C20 pad 1: Net-(U7B-+) -> Net-(U7A-+)
- C6 pad 1: Net-(U1B-+) -> Net-(U1A-+)
- C8 pad 1: Net-(U1B--) -> Net-(U1A--)
- JP_LIM1 pad 1: Net-(D1-A) -> Net-(JP_LIM1-A)
- R18 pad 1: Net-(U8-AINA) -> Net-(JP_LIM1-B)
- R6 pad 1: Net-(U1A--) -> Net-(U1B--)
- R6 pad 2: Net-(U1B-+) -> Net-(U1A-+)
- R7 pad 1: Net-(U1B--) -> Net-(U1A--)
- R8 pad 1: Net-(U1B--) -> Net-(U1A--)
- SW1 pad B: Net-(U6-C13) -> Net-(U6-C15)
- SW1 pad S2: Net-(U6-C15) -> /ROT.SW
- TP_LIM1 pad 1: Net-(D1-A) -> Net-(TP_LIM1-Pin_1)
- U1 pad 1: Net-(U1A--) -> Net-(C8-Pad2)
- U1 pad 3: /IN -> Net-(U1A-+)
- U1 pad 5: Net-(U1B-+) -> /IN
- U1 pad 7: Net-(C8-Pad2) -> Net-(U1B--)
- U5 pad 19: +5V -> Net-(U5-LEDA)
- U6 pad 10: unconnected-(U6-A15-Pad10) -> /LCD.RST
- U6 pad 11: unconnected-(U6-B3-Pad11) -> /LCD.CLK
- U6 pad 12: /BTN.PRE- -> unconnected-(U6-B4-Pad12)
- U6 pad 13: /BTN.PRE+ -> /LCD.DAT
- U6 pad 14: /BTN.VOL- -> /LCD.CS
- U6 pad 15: /BTN.VOL+ -> unconnected-(U6-B7-Pad15)
- U6 pad 16: /BTN.BNK- -> unconnected-(U6-B8-Pad16)
- U6 pad 17: /BTN.BNK+ -> unconnected-(U6-B9-Pad17)
- U6 pad 20: unconnected-(U6-3V3-Pad20) -> +3V3
- U6 pad 22: Net-(U6-C13) -> /BTN.BNK-
- U6 pad 28: unconnected-(U6-A2-Pad28) -> /BTN.PRE-
- U6 pad 29: /MCU.MCLK0 -> /BTN.PRE+
- U6 pad 30: /LCD.RST -> /BTN.VOL+
- U6 pad 31: /LCD.CLK -> /BTN.VOL-
- U6 pad 32: /LCD.CS -> /MCU.MCLK0
- U6 pad 33: /LCD.DAT -> unconnected-(U6-A7-Pad33)
- U6 pad 6: unconnected-(U6-A9-Pad6) -> /BTN.BNK+
- U6 pad 7: unconnected-(U6-A10-Pad7) -> /ROT.SW
- U6 pad 8: Net-(J3-D-) -> Net-(U6-USB_DM)
- U6 pad 9: Net-(J3-D+) -> Net-(U6-USB_DP)
- U7 pad 1: Net-(U7A--) -> /VREF_ADC
- U7 pad 2: Net-(U7A--) -> /VREF_ADC
- U7 pad 3: Net-(JP_LIM1-B) -> Net-(U7A-+)
- U7 pad 5: Net-(U7B-+) -> Net-(U7A-+)
- U7 pad 6: /VREF_ADC -> Net-(U7B--)
- U7 pad 7: /VREF_ADC -> Net-(U7B--)
- U8 pad 15: Net-(U7B-+) -> Net-(U7A-+)
- U8 pad 17: Net-(U8-AINA) -> Net-(JP_LIM1-B)
- U8 pad 18: Net-(U8-AINA) -> Net-(JP_LIM1-B)
- U8 pad 24: Net-(TP_OUT1-Pin_1) -> Net-(TP_OUT1-Pin_2)
- U8 pad 25: Net-(TP_OUT1-Pin_2) -> Net-(TP_OUT1-Pin_1)
Routing:
- net Net-(U6-C14): track 37.1 -> 148.2 mm, vias 0 -> 2
- net /ROT.SW: track 0.00 -> 97.6 mm
- net GNDREF: track 3.49 -> 96.6 mm, vias 0 -> 4
- net Net-(J3-D+): track 0.00 -> 89.0 mm
- net Net-(U6-C15): track 53.4 -> 142.1 mm, vias 0 -> 2
- net /LCD.CLK: track 0.00 -> 77.3 mm
- net Net-(J3-D-): track 0.00 -> 76.2 mm
- net /LCD.DAT: track 0.00 -> 75.2 mm
- net /LCD.CS: track 0.00 -> 74.9 mm
- net /BTN.PRE-: track 6.50 -> 70.2 mm
- net /BTN.VOL+: track 40.3 -> 97.9 mm
- net /LCD.RST: track 0.00 -> 51.7 mm
- net VCC: track 217.2 -> 268.9 mm, vias 6 -> 4
- net +3V3: track 53.6 -> 97.0 mm
- net Net-(U6-C13): track 36.1 -> 0.00 mm
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- added copper zone on F.Cu, net Net-(JP_LIM1-B)
- removed copper zone on F.Cu, net Net-(U8-AINA)
Other:
- board text added: "Multiefekt pedala v1.0 Lovro Zednik ${CURRENT_DATE}"
- board text added: "~{RST} DAC ADC CK LR"

Commit message: Prints and renders.
Parts:
- removed H1, H2, H3, H4: MountingHole_Pad, MountingHole:MountingHole_3.2mm_M3_Pad

Commit message: PCB work.
Parts:
- added C18: 68n, Capacitor_THT:C_Disc_D5.0mm_W2.5mm_P2.50mm, F.Cu at (171.0, 78.6)
- added H1: MountingHole_Pad, MountingHole:MountingHole_2.1mm, F.Cu at (46.8, 23.9)
- added H2: MountingHole_Pad, MountingHole:MountingHole_2.1mm, F.Cu at (134.8, 24.0)
- added H3: MountingHole_Pad, MountingHole:MountingHole_2.1mm, F.Cu at (46.7, 89.0)
- added H4: MountingHole_Pad, MountingHole:MountingHole_2.1mm, F.Cu at (134.8, 89.0)
- added H5: MountingHole_Pad, MountingHole:MountingHole_2.1mm, F.Cu at (48.2, 150.4)
- added H6: MountingHole_Pad, MountingHole:MountingHole_2.1mm, F.Cu at (226.2, 150.4)
- added H7: MountingHole_Pad, MountingHole:MountingHole_2.1mm, F.Cu at (226.2, 25.4)
- added R33: 100, Resistor_THT:R_Axial_DIN0207_L6.3mm_D2.5mm_P2.54mm_Vertical, F.Cu at (171.1, 73.4)
- C29: footprint Capacitor_THT:C_Disc_D5.0mm_W2.5mm_P5.00mm -> Capacitor_THT:C_Disc_D5.0mm_W2.5mm_P2.50mm
- R18: value 10k -> 100k
- moved TP_LIM1 31.8 mm to (199.8, 91.1)
- moved C1 13.3 mm to (181.9, 60.4)
- moved C32 4.94 mm to (198.0, 44.9)
- moved J3 4.80 mm to (56.0, 107.3)
- moved D2 4.41 mm to (163.6, 70.2), turned to 180 degrees
- moved D1 3.73 mm to (143.6, 66.9), turned to 90 degrees
- moved C12 3.61 mm to (174.2, 77.4), turned to 0 degrees
- moved JIN1 3.58 mm to (169.3, 34.1)
- moved R32 3.33 mm to (103.4, 71.5)
- moved JOUT1 2.94 mm to (216.8, 56.0)
- moved C31 2.56 mm to (140.8, 61.5)
- moved C29 2.41 mm to (167.8, 56.7), turned to 180 degrees
- moved C2 2.17 mm to (154.2, 45.3)
- moved U5 2.07 mm to (44.3, 91.5)
- moved R23 1.00 mm to (185.1, 109.1)
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Connections:
- C12 pad 1: Net-(TP_LIM1-Pin_1) -> Net-(C12-Pad1)
- R18 pad 1: Net-(JP_LIM1-B) -> Net-(JP_LIM1-A)
- TP_LIM1 pad 1: Net-(TP_LIM1-Pin_1) -> Net-(JP_LIM1-A)
- U1 pad 13: Net-(D1-A) -> Net-(D2-A)
- U1 pad 9: Net-(D1-A) -> Net-(D1-K)
- U4 pad 1: Net-(TP_LIM1-Pin_1) -> Net-(U4A--)
- U4 pad 2: Net-(TP_LIM1-Pin_1) -> Net-(U4A--)
Routing:
- net +3V3: track 97.0 -> 147.7 mm
- net Net-(TP_LIM1-Pin_1): track 16.6 -> 0.00 mm
- net GNDPWR: track 17.7 -> 28.9 mm, vias 0 -> 1
- net Net-(JP_LIM1-A): track 30.2 -> 39.3 mm
- net Net-(U4A--): track 0.00 -> 8.39 mm
- net Net-(C12-Pad1): track 0.00 -> 7.35 mm
- net Net-(JP_LIM1-B): track 16.2 -> 11.3 mm
- net Net-(U4B-+): track 15.0 -> 19.6 mm
- net Net-(U5-LEDA): track 9.18 -> 4.84 mm
- net Net-(J3-D+): track 89.0 -> 93.2 mm
- net Net-(J3-D-): track 76.2 -> 80.4 mm
- net Net-(D2-A): track 2.44 -> 6.01 mm
- net Net-(D1-K): track 2.40 -> 5.43 mm
- net Net-(U6-C14): track 148.2 -> 145.6 mm
- net /LCD.CS: track 74.9 -> 77.0 mm
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Other:
- board size 183 x 130 mm -> 188 x 135 mm
- copper layers 4 -> 2
