File: HW/zavrsni-h5-kicad/zavrsni-h5-kicad.kicad_pcb (KiCad board)
At the start: 2 copper layers, 83 parts, among them J1 DC Jack, J12V1 Conn_01x02, J12V_A1 Conn_01x02, J2 USB_B, J3 Conn_01x04, J3V3 Conn_01x02, J5V1 Conn_01x02, J5V_A1 Conn_01x02, SW1 EC11, U1 LM2596S-3.3, U2 AMS1117-5.0, U3 CS4272, U4 STM32H523CCU6, U5 TL072, U6 LM358, U7 TL072

Commit message: Počeo rad na završnoj tiskanoj pločici. Finaliziran odabran mikroupravljača (STM32H523CCU6). Postavljanje osnove routanja.
Parts:
- removed D2, D3: 1N4148W, Diode_SMD:D_SOD-123
- removed J12V1, J12V_A1, J3V3, J5V1, J5V_A1, JCDIN1: Conn_01x02, Connector_PinHeader_2.54mm:PinHeader_1x02_P2.54mm_Vertical
- removed J3: Conn_01x04, Connector_PinHeader_2.54mm:PinHeader_1x04_P2.54mm_Vertical
- removed R16, R19: 47k, Resistor_SMD:R_1206_3216Metric_Pad1.30x1.75mm_HandSolder
- removed R17, R18, R20: 5k1, Resistor_SMD:R_1206_3216Metric_Pad1.30x1.75mm_HandSolder
- removed SB12V1, SB3V3, SB5V1, SBCDIN1, SBGAIN1: SolderJumper_2_Open, Jumper:SolderJumper-2_P1.3mm_Open_TrianglePad1.0x1.5mm
- added J12VA1: Conn_01x02, Connector_PinHeader_2.54mm:PinHeader_1x02_P2.54mm_Vertical, B.Cu at (264.7, 104.1)
- added J12V_SB1: Conn_01x02, Connector_PinHeader_2.54mm:PinHeader_1x02_P2.54mm_Vertical, B.Cu at (269.3, 104.1)
- added J3V3_SB1: Conn_01x02, Connector_PinHeader_2.54mm:PinHeader_1x02_P2.54mm_Vertical, F.Cu at (124.5, 91.0)
- added J5VA1: Conn_01x02, Connector_PinHeader_2.54mm:PinHeader_1x02_P2.54mm_Vertical, B.Cu at (273.9, 104.1)
- added J5V_SB1: Conn_01x02, Connector_PinHeader_2.54mm:PinHeader_1x02_P2.54mm_Vertical, B.Cu at (278.5, 104.1)
- added JCDIN_SB1: Conn_01x02, Connector_PinHeader_2.54mm:PinHeader_1x02_P2.54mm_Vertical, B.Cu at (283.1, 104.1)
- added JGAIN_SB1: Conn_01x02, Jumper:SolderJumper-2_P1.3mm_Open_TrianglePad1.0x1.5mm, B.Cu at (281.3, 147.8)
- added JUART1: Conn_01x03, Connector_PinHeader_2.54mm:PinHeader_1x03_P2.54mm_Vertical, F.Cu at (146.5, 68.3)
- added R32: 150, Resistor_THT:R_Axial_DIN0411_L9.9mm_D3.6mm_P12.70mm_Horizontal, B.Cu at (264.4, 96.7)
- C12, C13, C14, C15, C16, C17, C18, C19, C2, C20, C21, C22, C23, C24, C26, C27, C28, C29, C30, C31, C32, C33, C34, C35, C36, C37, C8, D1, D4, J1, J2, JIN1, JOUT1, L1, R12, R13, R15, R2, R21, R22, R23, R24, R25, R26, R27, R28, R29, R3, R30, R4, R5, R6, SW1, U1, U2, U5, U6, U7: moved to B.Cu
- C25: value 220p -> 1n; moved to B.Cu
- R14: value 47k -> 10k; moved to B.Cu
- moved D4 142.9 mm to (279.0, 135.8)
- moved JIN1 113.5 mm to (238.4, 146.9)
- moved JOUT1 104.2 mm to (238.4, 130.9)
- moved JCD1 96.4 mm to (152.8, 63.1), turned to 180 degrees
- moved U8 95.0 mm to (23.9, 93.5)
- moved C2 90.7 mm to (123.0, 82.4), turned to 90 degrees
- moved C37 90.3 mm to (258.2, 93.7)
- moved U4 90.0 mm to (133.8, 58.1)
- moved C8 85.1 mm to (129.8, 82.2), turned to 90 degrees
- moved C36 84.6 mm to (258.2, 100.2)
- moved C21 82.3 mm to (177.2, 45.8), turned to 180 degrees
- moved R6 80.8 mm to (259.6, 153.4)
- moved R26 80.7 mm to (271.5, 153.4)
- moved C33 80.5 mm to (258.2, 106.8)
- moved R13 78.9 mm to (259.6, 146.8)
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Connections:
- net /CODEC_SDIN renamed /CODEC_MOSI
- net /CODEC_SDOUT renamed /CODEC_MISO
- C25 pad 1: Net-(U5A-+) -> Net-(C25-Pad1)
- C26 pad 1: Net-(C26-Pad1) -> Net-(C25-Pad1)
- R14 pad 2: Net-(U5A-+) -> Net-(C25-Pad1)
- R2 pad 1: unconnected-(R2-Pad1) -> Net-(U4-A5)
- R21 pad 2: Net-(U7A-+) -> Net-(U5A-+)
- R22 pad 2: Net-(U7A--) -> Net-(U5A--)
- R23 pad 1: Net-(U7A--) -> Net-(U5A--)
- R3 pad 1: unconnected-(R3-Pad1) -> Net-(U4-A7)
- R30 pad 1: Net-(U7A-+) -> Net-(U5A-+)
- R4 pad 1: unconnected-(R4-Pad1) -> Net-(U4-A6)
- R5 pad 1: unconnected-(R5-Pad1) -> Net-(U4-A3)
- R6 pad 2: Net-(U7A-+) -> Net-(U5A-+)
- U4 pad 14: unconnected-(U4-B6-Pad14) -> /CODEC_SCL
- U4 pad 15: unconnected-(U4-B7-Pad15) -> /CODEC_SDA
- U4 pad 16: unconnected-(U4-B8-Pad16) -> /CODEC_RST
- U4 pad 26: unconnected-(U4-A0-Pad26) -> /U_TX
- U4 pad 27: unconnected-(U4-A1-Pad27) -> /U_RX
- U4 pad 29: unconnected-(U4-A3-Pad29) -> Net-(U4-A3)
- U4 pad 3: unconnected-(U4-B14-Pad3) -> /LCD.CS
- U4 pad 30: unconnected-(U4-A4-Pad30) -> /CODEC_WS
- U4 pad 31: unconnected-(U4-A5-Pad31) -> Net-(U4-A5)
- U4 pad 32: unconnected-(U4-A6-Pad32) -> Net-(U4-A6)
- U4 pad 33: unconnected-(U4-A7-Pad33) -> Net-(U4-A7)
- U4 pad 38: +3V3 -> unconnected-(U4-3V3-Pad38)
- U4 pad 4: unconnected-(U4-B15-Pad4) -> /LCD.DAT
- U4 pad 6: unconnected-(U4-A9-Pad6) -> /LCD.CLK
- U4 pad 7: unconnected-(U4-A10-Pad7) -> /LCD.RST
- U5 pad 1: Net-(U5A--) -> Net-(C30-Pad1)
- U6 pad 1: Net-(D2-K) -> (no net)
- U6 pad 2: Net-(D2-K) -> (no net)
- U6 pad 3: Net-(U6A-+) -> (no net)
- U6 pad 5: Net-(U6B-+) -> (no net)
- U6 pad 6: Net-(D3-A) -> (no net)
- U6 pad 7: Net-(D3-A) -> (no net)
- U7 pad 1: Net-(C30-Pad1) -> (no net)
- U7 pad 2: Net-(U7A--) -> (no net)
- U7 pad 3: Net-(U7A-+) -> (no net)
- U7 pad 5: unconnected-(U7B-+-Pad5) -> (no net)
- U7 pad 6: unconnected-(U7B---Pad6) -> (no net)
- U7 pad 7: unconnected-(U7-Pad7) -> (no net)
- U8 pad 1: unconnected-(U8-GND-Pad1) -> GNDPWR
- U8 pad 15: unconnected-(U8-PSB-Pad15) -> GNDPWR
- U8 pad 17: unconnected-(U8-~{RST}-Pad17) -> /LCD.RST
- U8 pad 19: unconnected-(U8-LEDA-Pad19) -> Net-(U8-LEDA)
- U8 pad 2: unconnected-(U8-VCC-Pad2) -> +3V3
- U8 pad 20: unconnected-(U8-LEDK-Pad20) -> GNDPWR
- U8 pad 4: unconnected-(U8-RS-Pad4) -> /LCD.CS
- U8 pad 5: unconnected-(U8-R/W-Pad5) -> /LCD.DAT
- U8 pad 6: unconnected-(U8-E-Pad6) -> /LCD.CLK
Routing:
- net /LCD.CS: track 0.00 -> 122.0 mm
- net /LCD.DAT: track 0.00 -> 118.4 mm
- net +3V3: track 0.00 -> 113.4 mm
- net /LCD.CLK: track 0.00 -> 113.2 mm
- net /CODEC_RST: track 0.00 -> 97.9 mm
- net /CODEC_SDA: track 0.00 -> 93.6 mm
- net /CODEC_SCL: track 0.00 -> 90.3 mm
- net /LCD.RST: track 0.00 -> 84.4 mm
- net /CODEC_MOSI: track 0.00 -> 38.5 mm
- net /CODEC_MISO: track 0.00 -> 33.5 mm
- net /CODEC_WS: track 0.00 -> 31.6 mm
- net /CODEC_SCLK: track 0.00 -> 28.8 mm
- net /CODEC_MCK: track 0.00 -> 19.5 mm
- net +12V: track 0.00 -> 6.70 mm
- net Net-(U3-FILT+): track 0.00 -> 6.61 mm
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- added copper zone on B.Cu, net +3V3
- added copper zone on B.Cu, net /CODEC_IN
- added copper zone on B.Cu, net GNDPWR
- added copper zone on F.Cu, net GNDPWR
- added copper zone on B.Cu, net Net-(D1-K)
- added copper zone on B.Cu, net Net-(J3V3_SB1-Pin_1)
