File: HW/zavrsni-h5-kicad/zavrsni-h5-kicad.kicad_sch (KiCad schematic)
At the start: 82 parts, among them J1 DC Jack, J12V1 Conn_01x02, J12V_A1 Conn_01x02, J2 USB_B, J3 Conn_01x04, J3V3 Conn_01x02, J5V1 Conn_01x02, J5V_A1 Conn_01x02, SW1 EC11, U1 LM2596S-3.3, U2 AMS1117-5.0, U3 CS4272, U4 STM32H523CCU6, U5 TL072, U6 LM358, U7 TL072

Commit message: Počeo rad na završnoj tiskanoj pločici. Finaliziran odabran mikroupravljača (STM32H523CCU6). Postavljanje osnove routanja.
Parts:
- removed D2, D3: 1N4148W, Diode_SMD:D_SOD-123, symbol Diode:1N4148W
- removed J12V1, J12V_A1, J3V3, J5V1, JCDIN1: Conn_01x02, Connector_PinHeader_2.54mm:PinHeader_1x02_P2.54mm_Vertical, symbol Connector_Generic:Conn_01x02
- removed J3: Conn_01x04, Connector_PinHeader_2.54mm:PinHeader_1x04_P2.54mm_Vertical, symbol Connector_Generic:Conn_01x04
- removed R16, R19: 47k, Resistor_SMD:R_1206_3216Metric_Pad1.30x1.75mm_HandSolder, symbol Device:R
- removed R17, R18: 5k1, Resistor_SMD:R_1206_3216Metric_Pad1.30x1.75mm_HandSolder, symbol Device:R
- removed SB5V1: SolderJumper_2_Open, Jumper:SolderJumper-2_P1.3mm_Open_TrianglePad1.0x1.5mm, symbol Jumper:SolderJumper_2_Open
- removed unit 2 of U6
- removed unit 1 of U6
- added J12VA1, J5V_SB1: Conn_01x02, Connector_PinHeader_2.54mm:PinHeader_1x02_P2.54mm_Vertical, symbol Connector_Generic:Conn_01x02
- added JUART1: Conn_01x03, Connector_PinHeader_2.54mm:PinHeader_1x03_P2.54mm_Vertical, symbol Connector_Generic:Conn_01x03
- added R32: 150, Resistor_THT:R_Axial_DIN0411_L9.9mm_D3.6mm_P12.70mm_Horizontal, symbol Device:R
- J12V_SB1: renamed from SB12V1; value SolderJumper_2_Open -> Conn_01x02; footprint Jumper:SolderJumper-2_P1.3mm_Open_TrianglePad1.0x1.5mm -> Connector_PinHeader_2.54mm:PinHeader_1x02_P2.54mm_Vertical; symbol Jumper:SolderJumper_2_Open -> Connector_Generic:Conn_01x02; now in the parts list
- J2: now not fitted
- J3V3_SB1: renamed from SB3V3; value SolderJumper_2_Open -> Conn_01x02; footprint Jumper:SolderJumper-2_P1.3mm_Open_TrianglePad1.0x1.5mm -> Connector_PinHeader_2.54mm:PinHeader_1x02_P2.54mm_Vertical; symbol Jumper:SolderJumper_2_Open -> Connector_Generic:Conn_01x02; now in the parts list
- JCDIN_SB1: renamed from SBCDIN1; value SolderJumper_2_Open -> Conn_01x02; footprint Jumper:SolderJumper-2_P1.3mm_Open_TrianglePad1.0x1.5mm -> Connector_PinHeader_2.54mm:PinHeader_1x02_P2.54mm_Vertical; symbol Jumper:SolderJumper_2_Open -> Connector_Generic:Conn_01x02; now in the parts list
- JGAIN_SB1: renamed from SBGAIN1; value SolderJumper_2_Open -> Conn_01x02; symbol Jumper:SolderJumper_2_Open -> Connector_Generic:Conn_01x02; now in the parts list
- renumbered J5V_A1 to J5VA1
Connections:
- net +12V_A: now also J12VA1.1 (Pin_1), J12VA1.2 (Pin_2)
- net +3V3: now also U8.2 (VCC); no longer U4.38 (3V3)
- net +5V: now also J5V_SB1.2 (Pin_2)
- net CODEC_RST: now also U4.16 (B8)
- net CODEC_SCL: now also U4.14 (B6)
- net CODEC_SDA: now also U4.15 (B7)
- net CODEC_WS: now also U4.30 (A4)
- net GNDPWR: now also U8.1 (GND), U8.15 (PSB), U8.20 (LEDK), JUART1.3 (Pin_3)
- net at C15.1, C33.1, U2.2 (VO): now also J5V_SB1.1 (Pin_1)
- net at R2.1: now also U4.31 (A5)
- net LCD.RST: now reaches U8.17 (~{RST})
- net LCD.RST: now also U4.7 (A10)
- net at U8.19 (LEDA): now also R32.2
- net LCD.CS: now reaches U8.4 (RS)
- net LCD.CS: now also U4.3 (B14)
- net LCD.DAT: now reaches U8.5 (R/W)
- net LCD.DAT: now also U4.4 (B15)
- net LCD.CLK: now reaches U8.6 (E)
- net LCD.CLK: now also U4.6 (A9)
- net U_TX: now reaches U4.26 (A0)
- net U_TX: now also JUART1.2 (Pin_2)
- net U_RX: now reaches U4.27 (A1)
- net U_RX: now also JUART1.1 (Pin_1)
- net at U4.29 (A3): now also R5.1
- net at U4.32 (A6): now also R4.1
- net at U4.33 (A7): now also R3.1
- net CODEC_SDIN renamed CODEC_MOSI
- net CODEC_SDOUT renamed CODEC_MISO
- new net VCC: R32.1
- no-connect marks 10 -> 21
Other:
- moved on the sheet: C2, C23, C36, C37, C8, J12V_SB1, J3V3_SB1, J5VA1, JCDIN_SB1, JGAIN_SB1, R13, R2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
